File: IFS08-MainLite/MAIN_LITE.kicad_sch (KiCad schematic)
At the start: 79 parts, among them IC1 BMI088, J1 Micro_SD_Card_Det1, J2 Conn_01x04_Socket, J3 Conn_01x18_Pin, J4 Conn_01x18_Pin, J5 USB_C_Receptacle_USB2.0_14P, SW1 SW_Push, SW2 SW_Push, U1 LD39200PU33R, U2 TCAN330, U3 TCAN330, U4 TCAN330, U5 STM32H733ZGTx, Y1 24MHz

Commit message: fix(hw): make schematic ERC-clean and fail CI on ERC errors
- Add no-connect flags to the 53 unwired STM32 pins that ERC reported
  (pin_not_connected).
- Add PWR_FLAGs on GND, +3V3/VDD and +5V (power_pin_not_driven: the
  LD39200 output and the backplane +5V have no power-output pin type).
- Remove two dangling no-connect flags (one placed off-sheet).
- Set ERC_BLOCKING to true; re-export the schematic PDF.

Connectivity is unchanged: the netlist is identical; the pin model only
changes in no_connect_flag and schematic_git_blob.
Connections:
- no-connect marks 31 -> 82
